File: noise-and-ring-modulator-v1.0.sch (EAGLE design)
At the start: 71 parts, among them IC1 TL074JT, IC2 TL072JT, T1 NOISE-2N3904, U1 MC1496DR2G

Commit message: Tiny silk screen fix
Other:
- note added: "+12V"
- note added: "-12V"
- note removed: "+15V"
- note removed: "-15V"
Changed lines of the file:
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@@
 <wire x1="17.78" y1="109.22" x2="17.78" y2="104.14" width="0.1524" layer="97"/>
 <text x="17.78" y="111.76" size="1.778" layer="97">470 / 500R</text>
-<text x="10.16" y="119.38" size="1.778" layer="97">+15V</text>
+<text x="10.16" y="119.38" size="1.778" layer="97">+12V</text>
 <wire x1="17.78" y1="27.94" x2="12.7" y2="27.94" width="0.1524" layer="97"/>
 <wire x1="15.24" y1="25.4" x2="12.7" y2="27.94" width="0.1524" layer="97"/>
@@
 <wire x1="7.62" y1="27.94" x2="7.62" y2="33.02" width="0.1524" layer="97"/>
 <text x="17.78" y="22.86" size="1.778" layer="97">200 / 220R</text>
-<text x="15.24" y="17.78" size="1.778" layer="97" rot="R180">-15V</text>
+<text x="15.24" y="17.78" size="1.778" layer="97" rot="R180">-12V</text>
 <text x="-53.34" y="66.04" size="1.778" layer="97">DC inputs, add 1uF
 series caps for AC</text>

Commit message: Replaced pin footprints
Parts:
- removed PINK, RED, WHITE, X1, X10, X2, X20, X21, X22, X3, X4, X5, X6, X7, X8, X9: (no value), joakim:MA01-1JN
- added X11, X12: (no value), joakim:MA08-1JN
Connections:
- net +12V: now also X12.8; no longer X1.1
- net -12V: now also X11.1; no longer X3.1
- net CARRIER: now also X12.4; no longer X7.1
- net CAR_TRIM_1: now also X12.3; no longer X9.1
- net CAR_TRIM_2: now also X12.2; no longer X8.1
- net GND: now also X12.5; no longer X2.1
- net LEV1: now also X11.3; no longer X20.1
- net LEV2: now also X11.2; no longer X22.1
- net OUT: now also X12.1; no longer X10.1
- net PINK: now also X12.6; no longer PINK.1
- net RED: now also X11.4; no longer RED.1
- net SIGNAL: now also X11.7; no longer X6.1
- net SIG_TRIM_1: now also X11.6; no longer X5.1
- net SIG_TRIM_2: now also X11.5; no longer X4.1
- net WHITE: now also X12.7; no longer WHITE.1
Other:
- moved on the sheet: R22
