File: distortion-noise-and-ring-modulator-v1.0.brd (EAGLE design)
At the start: 44.8 x 17.8 mm, 72 parts, among them IC1 TL074JT, IC4 LM13700SL, IC5 TL074JT, Q1 MMBT3906, T1 NOISE-2N3904, U1 MC1496DR2G

Commit message: Added bom and checked parts and pcb with JLCPCB
Parts:
- C1: device rcl:UD-4X5,8_NICHICON -> rcl:E2-5
- moved C1 0.32 mm to (39.7, 15.2), turned to 0 degrees
Other:
- outline, holes or cut-outs redrawn
Changed lines of the file:
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@@
 <setting verticaltext="up"/>
 </settings>
-<grid distance="12.5" unitdist="mil" unit="mil" style="lines" multiple="1" display="yes" altdistance="0.025" altunitdist="inch" altunit="inch"/>
+<grid distance="50" unitdist="mil" unit="mil" style="lines" multiple="1" display="yes" altdistance="0.025" altunitdist="inch" altunit="inch"/>
 <layers>
 <layer number="1" name="Top" color="4" fill="1" visible="yes" active="yes"/>
@@
 <layer number="23" name="tOrigins" color="15" fill="1" visible="yes" active="yes"/>
 <layer number="24" name="bOrigins" color="15" fill="1" visible="no" active="yes"/>
-<layer number="25" name="tNames" color="7" fill="1" visible="no" active="yes"/>
-<layer number="26" name="bNames" color="7" fill="1" visible="no" active="yes"/>
+<layer number="25" name="tNames" color="7" fill="1" visible="yes" active="yes"/>
+<layer number="26" name="bNames" color="7" fill="1" visible="yes" active="yes"/>
 <layer number="27" name="tValues" color="7" fill="1" visible="no" active="yes"/>
 <layer number="28" name="bValues" color="7" fill="1" visible="no" active="yes"/>
@@
 <board>
 <plain>
-<wire x1="0" y1="0" x2="44.7675" y2="0" width="0" layer="20"/>
+<wire x1="1.27" y1="0" x2="44.7675" y2="0" width="0" layer="20"/>
 <wire x1="44.7675" y1="0" x2="44.7675" y2="17.78" width="0" layer="20"/>
 <wire x1="44.7675" y1="17.78" x2="0" y2="17.78" width="0" layer="20"/>
-<wire x1="0" y1="17.78" x2="0" y2="0" width="0" layer="20"/>
+<wire x1="0" y1="17.78" x2="0" y2="1.27" width="0" layer="20"/>
+<wire x1="0" y1="1.27" x2="1.27" y2="0" width="0" layer="20"/>
 <text x="8.255" y="15.24" size="1.27" layer="26" font="vector" rot="MR270">+12v</text>
 <text x="6.985" y="2.8575" size="1.27" layer="26" font="vector" rot="MR90">-12v</text>
@@
 <wire x1="21.59" y1="13.97" x2="22.86" y2="13.97" width="0.1016" layer="26"/>
 <text x="31.115" y="0.3175" size="0.6096" layer="25" font="vector" rot="R90">4VOB</text>
-<text x="41.5925" y="16.1925" size="1.778" layer="26" font="vector" rot="MR270">Ring mod,
+<text x="37.465" y="16.1925" size="1.778" layer="26" font="vector" rot="MR270">Ring mod,
 distortion
 &amp; Noise</text>
@@
 <attribute name="VALUE" x="24.13" y="14.605" size="1.27" layer="27" rot="R270"/>
 </element>
-<element name="C1" library="rcl" library_urn="urn:adsk.eagle:library:334" package="UD-4X5,8_NICHICON" package3d_urn="urn:adsk.eagle:package:23474/1" value="100u 25V" x="39.37" y="15.24" smashed="yes" rot="R180">
-<attribute name="NAME" x="42.8625" y="17.145" size="0.6096" layer="25" font="vector" rot="R180"/>
-<attribute name="POPULARITY" value="0" x="39.37" y="15.24" size="1.778" layer="27" rot="R180" display="off"/>
-<attribute name="SPICEPREFIX" value="C" x="39.37" y="15.24" size="1.778" layer="27" rot="R180" display="off"/>
-<attribute name="VALUE" x="41.275" y="18.415" size="1.016" layer="27" rot="R180"/>
+<element name="C1" library="rcl" library_urn="urn:adsk.eagle:library:334" package="E2-5" package3d_urn="urn:adsk.eagle:package:23346/2" value="100u 25V" x="39.6875" y="15.24" smashed="yes">
+<attribute name="NAME" x="42.2275" y="16.8275" size="0.6096" layer="25" font="vector"/>
+<attribute name="POPULARITY" value="14" x="39.6875" y="15.24" size="1.778" layer="27" display="off"/>
+<attribute name="SPICEPREFIX" value="C" x="39.6875" y="15.24" size="1.778" layer="27" display="off"/>
+<attribute name="VALUE" x="37.7825" y="12.065" size="1.016" layer="27"/>
 </element>
 <element name="R13" library="rcl" library_urn="urn:adsk.eagle:library:334" package="R0402" package3d_urn="urn:adsk.eagle:package:23547/3" value="6k8" x="24.13" y="3.81" smashed="yes" rot="R90">
@@
 </element>
 <element name="C15" library="joakim" package="C0402-J" value="100nF" x="43.18" y="13.97" smashed="yes" rot="R180">
-<attribute name="NAME" x="42.2275" y="14.605" size="0.6096" layer="25" font="vector"/>
+<attribute name="NAME" x="42.545" y="14.605" size="0.6096" layer="25" font="vector"/>
 <attribute name="VALUE" x="43.815" y="15.875" size="1.27" layer="27" rot="R180"/>
 </element>
@@
 <wire x1="27.305" y1="13.47" x2="27.305" y2="12.7" width="0.254" layer="1"/>
 <via x="27.305" y="12.7" extent="1-16" drill="0.3302"/>
-<wire x1="42.2275" y1="15.24" x2="40.795" y2="15.24" width="0.254" layer="1"/>
+<wire x1="42.2275" y1="15.24" x2="40.7035" y2="15.24" width="0.254" layer="1"/>
 <via x="42.2275" y="15.24" extent="1-16" drill="0.3302"/>
 <wire x1="30.48" y1="3.31" x2="30.48" y2="2.9925" width="0.254" layer="1"/>
@@
 <wire x1="23.8125" y1="14.9225" x2="21.9075" y2="14.9225" width="0.254" layer="16"/>
 <wire x1="23.8125" y1="14.9225" x2="24.13" y2="15.24" width="0.254" layer="16"/>
-<wire x1="37.945" y1="15.24" x2="37.945" y2="14.605" width="0.254" layer="1"/>
-<wire x1="37.945" y1="14.605" x2="37.6275" y2="14.2875" width="0.254" layer="1"/>
+<wire x1="38.6715" y1="15.24" x2="38.4175" y2="14.76" width="0.254" layer="1"/>
+<wire x1="38.4175" y1="14.76" x2="36.9925" y2="13.335" width="0.254" layer="1"/>
 <wire x1="24.765" y1="14.47" x2="24.765" y2="15.24" width="0.254" layer="1"/>
-<wire x1="37.6275" y1="14.2875" x2="37.6275" y2="13.97" width="0.254" layer="16"/>
-<wire x1="37.6275" y1="13.97" x2="36.04" y2="12.3825" width="0.254" layer="16"/>
+<wire x1="36.9925" y1="13.335" x2="36.04" y2="12.3825" width="0.254" layer="16"/>
 <wire x1="36.04" y1="12.3825" x2="32.865" y2="12.3825" width="0.254" layer="16"/>
 <wire x1="32.865" y1="12.3825" x2="30.6425" y2="14.605" width="0.254" layer="16"/>
@@
 <wire x1="27.305" y1="14.605" x2="26.67" y2="15.24" width="0.254" layer="16"/>
 <via x="26.67" y="15.24" extent="1-16" drill="0.3302"/>
-<via x="37.6275" y="14.2875" extent="1-16" drill="0.3302"/>
+<via x="36.9925" y="13.335" extent="1-16" drill="0.3302"/>
 </signal>
 <signal name="N$11">
