File: distortion-noise-and-ring-modulator-v1.0.sch (EAGLE design)
At the start: 72 parts, among them IC1 TL074JT, IC4 LM13700SL, IC5 TL074JT, Q1 MMBT3906, T1 NOISE-2N3904, U1 MC1496DR2G

Commit message: Added bom and checked parts and pcb with JLCPCB
Parts:
- C1: device rcl:CPOL-EUUD-4X5,8 -> rcl:CPOL-EUE2-5
Other:
- note added: "TODO: Simulate 3k3 instead of 3k here"
Changed lines of the file:
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@@
 <part name="R1" library="rcl" library_urn="urn:adsk.eagle:library:334" deviceset="R-EU_" device="R0402" package3d_urn="urn:adsk.eagle:package:23547/3" value="1k5"/>
 <part name="R19" library="rcl" library_urn="urn:adsk.eagle:library:334" deviceset="R-EU_" device="R0402" package3d_urn="urn:adsk.eagle:package:23547/3" value="1k5"/>
-<part name="C1" library="rcl" library_urn="urn:adsk.eagle:library:334" deviceset="CPOL-EU" device="UD-4X5,8" package3d_urn="urn:adsk.eagle:package:23474/1" value="100u 25V"/>
+<part name="C1" library="rcl" library_urn="urn:adsk.eagle:library:334" deviceset="CPOL-EU" device="E2-5" package3d_urn="urn:adsk.eagle:package:23346/2" value="100u 25V"/>
 <part name="GND3" library="supply1" library_urn="urn:adsk.eagle:library:371" deviceset="GND" device=""/>
 <part name="R13" library="rcl" library_urn="urn:adsk.eagle:library:334" deviceset="R-EU_" device="R0402" package3d_urn="urn:adsk.eagle:package:23547/3" value="6k8"/>
@@
 not available as
 C0G in 0603 or 0402</text>
+<text x="60.96" y="48.26" size="1.778" layer="91">TODO: Simulate 3k3 instead of 3k here</text>
 </plain>
 <instances>
