File: distortion-noise-and-ring-modulator-v1.1.brd (EAGLE design)
At the start: 44.8 x 24.1 mm, 75 parts, among them IC1 TL074JT, IC2 TL074JT, IC3 LM13700SL, Q1 MMBT3906, T1 NOISE-2N3904, U1 MC1496DR2G, X1 MA06-1JN, X2 MA06-1JN

Commit message: V1.1 ready for production
Parts:
- T1: value NOISE-2N3904 -> NOISE-2N3904-DNM
- X1, X2: value MA06-1JN -> MA06-1JN-DNM
Changed lines of the file:
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@@
 <attribute name="VALUE" x="6.35" y="10.16" size="1.27" layer="27"/>
 </element>
-<element name="T1" library="joakim" package="NOISE-2N3904-J" value="NOISE-2N3904" x="2.8575" y="4.7625" smashed="yes" rot="R180">
+<element name="T1" library="joakim" package="NOISE-2N3904-J" value="NOISE-2N3904-DNM" x="2.8575" y="4.7625" smashed="yes" rot="R180">
 <attribute name="NAME" x="5.23875" y="6.38175" size="0.6096" layer="25" font="vector"/>
 <attribute name="VALUE" x="5.3975" y="8.0645" size="1.27" layer="27" ratio="10" rot="R180"/>
@@
 <attribute name="VALUE" x="29.155" y="-2.045" size="1.27" layer="27"/>
 </element>
-<element name="X1" library="joakim" package="MA06N-1J" value="MA06-1JN" x="21.59" y="3.81" smashed="yes">
+<element name="X1" library="joakim" package="MA06N-1J" value="MA06-1JN-DNM" x="21.59" y="3.81" smashed="yes">
 <attribute name="VALUE" x="17.78" y="0.889" size="1.27" layer="27" ratio="10"/>
 </element>
-<element name="X2" library="joakim" package="MA06N-1J" value="MA06-1JN" x="21.59" y="19.05" smashed="yes" rot="R180">
+<element name="X2" library="joakim" package="MA06N-1J" value="MA06-1JN-DNM" x="21.59" y="19.05" smashed="yes" rot="R180">
 <attribute name="VALUE" x="25.4" y="21.971" size="1.27" layer="27" ratio="10" rot="R180"/>
 </element>
